Commit message: [kobuki_description] started ros2 conversion
Install all dirs and declare ament package

Building kobuki_description with ros2

update imu plugin

xacro prefix to get rid of deprecation warning

Use differential drive controller for base in gazebo

Fix base_footprint parenting to base_link

Include imu plugin

WIP closer to kobuki_ros

Signed-off-by: Emerson Knapp <emerson.b.knapp@gmail.com>

File: kobuki_description/urdf/kobuki.urdf.xacro (robot description, xacro)
@@ -23,6 +23,6 @@
     <joint name="base_joint" type="fixed">
       <origin xyz="0 0 0.0102" rpy="0 0 0" />
-      <parent link="base_footprint"/>
-      <child link="base_link" />
+      <parent link="base_link"/>
+      <child link="base_footprint" />
     </joint>
     <link name="base_link">
@@ -209,5 +209,5 @@
     </link>
     <!-- Kobuki Gazebo simulation details -->
-    <kobuki_sim/>
+    <xacro:kobuki_sim/>
   </xacro:macro>
 </robot>

File: kobuki_description/urdf/kobuki_gazebo.urdf.xacro (robot description, xacro)
@@ -138,4 +138,12 @@
 	  <gazebo reference="gyro_link">
 	   <sensor type="imu" name="imu">
+        <plugin name="gazebo_ros_imu_controller" filename="libgazebo_ros_imu_sensor.so">
+          <ros>
+            <argument>~/out:=imu</argument>
+          </ros>
+          <output_type>sensor_msgs/msg/Imu</output_type>
+          <body_name>gyro_link</body_name>
+          <frame_name>gyro_link</frame_name>
+        </plugin>
         <always_on>true</always_on>
         <update_rate>50</update_rate>
@@ -161,18 +169,20 @@
 	  </gazebo>
 	  <gazebo>
-	    <plugin name="kobuki_controller" filename="libgazebo_ros_kobuki.so">
-	      <publish_tf>1</publish_tf>
-	      <left_wheel_joint_name>wheel_left_joint</left_wheel_joint_name>
-	      <right_wheel_joint_name>wheel_right_joint</right_wheel_joint_name>
-	      <wheel_separation>.230</wheel_separation>
-	      <wheel_diameter>0.070</wheel_diameter>
-	      <torque>1.0</torque>
-	      <velocity_command_timeout>0.6</velocity_command_timeout>
-	      <cliff_sensor_left_name>cliff_sensor_left</cliff_sensor_left_name>
-	      <cliff_sensor_center_name>cliff_sensor_front</cliff_sensor_center_name>
-	      <cliff_sensor_right_name>cliff_sensor_right</cliff_sensor_right_name>
-	      <cliff_detection_threshold>0.04</cliff_detection_threshold>
-	      <bumper_name>bumpers</bumper_name>
-        <imu_name>imu</imu_name>
+	    <plugin name="differential_drive_controller" filename="libgazebo_ros_diff_drive.so">
+    		<update_rate>10</update_rate>
+        <left_joint>wheel_left_joint</left_joint>
+        <right_joint>wheel_right_joint</right_joint>
+        <wheel_separation>0.230</wheel_separation>
+        <wheel_diameter>0.070</wheel_diameter>
+        <max_wheel_torque>1.0</max_wheel_torque>
+        <max_wheel_acceleration>1.0</max_wheel_acceleration>
+        <command_topic>cmd_vel</command_topic>
+        <!-- output -->
+        <publish_odom>true</publish_odom>
+        <publish_odom_tf>true</publish_odom_tf>
+        <publish_wheel_tf>true</publish_wheel_tf>
+        <odometry_topic>odom</odometry_topic>
+        <odometry_frame>odom</odometry_frame>
+        <robot_base_frame>base_link</robot_base_frame>
 	    </plugin>
 	  </gazebo>

Commit message: Fix base_footprint parenting to base_link

File: kobuki_description/urdf/kobuki.urdf.xacro (robot description, xacro)
@@ -11,19 +11,4 @@
   <!-- Kobuki -->
   <xacro:macro name="kobuki">
-    <link name="base_footprint"/>
-    <!--
-       Base link is set at the bottom of the base mould.
-       This is done to be compatible with the way base link
-       was configured for turtlebot 1. Refer to
-       https://github.com/turtlebot/turtlebot/issues/40
-       To put the base link at the more oft used wheel
-       axis, set the z-distance from the base_footprint
-       to 0.352.
-      -->
-    <joint name="base_joint" type="fixed">
-      <origin xyz="0 0 0.0102" rpy="0 0 0" />
-      <parent link="base_footprint"/>
-      <child link="base_link" />
-    </joint>
     <link name="base_link">
       <visual>
@@ -56,4 +41,19 @@
       </inertial>
     </link>
+    <link name="base_footprint"/>
+    <!--
+       Base link is set at the bottom of the base mould.
+       This is done to be compatible with the way base link
+       was configured for turtlebot 1. Refer to
+       https://github.com/turtlebot/turtlebot/issues/40
+       To put the base link at the more oft used wheel
+       axis, set the z-distance from the base_footprint
+       to 0.352.
+      -->
+    <joint name="base_joint" type="fixed">
+      <origin xyz="0 0 0.0102" rpy="0 0 0" />
+      <parent link="base_link"/>
+      <child link="base_footprint" />
+    </joint>
     <joint name="wheel_left_joint" type="continuous">
       <parent link="base_link"/>

Commit message: WIP closer to kobuki_ros
Signed-off-by: Emerson Knapp <emerson.b.knapp@gmail.com>

File: kobuki_description/urdf/kobuki.urdf.xacro (robot description, xacro)
@@ -11,4 +11,19 @@
   <!-- Kobuki -->
   <xacro:macro name="kobuki">
+    <link name="base_footprint"/>
+    <!--
+       Base link is set at the bottom of the base mould.
+       This is done to be compatible with the way base link
+       was configured for turtlebot 1. Refer to
+       https://github.com/turtlebot/turtlebot/issues/40
+       To put the base link at the more oft used wheel
+       axis, set the z-distance from the base_footprint
+       to 0.352.
+      -->
+    <joint name="base_joint" type="fixed">
+      <origin xyz="0 0 0.0102" rpy="0 0 0" />
+      <parent link="base_link"/>
+      <child link="base_footprint" />
+    </joint>
     <link name="base_link">
       <visual>
@@ -41,19 +56,4 @@
       </inertial>
     </link>
-    <link name="base_footprint"/>
-    <!--
-       Base link is set at the bottom of the base mould.
-       This is done to be compatible with the way base link
-       was configured for turtlebot 1. Refer to
-       https://github.com/turtlebot/turtlebot/issues/40
-       To put the base link at the more oft used wheel
-       axis, set the z-distance from the base_footprint
-       to 0.352.
-      -->
-    <joint name="base_joint" type="fixed">
-      <origin xyz="0 0 0.0102" rpy="0 0 0" />
-      <parent link="base_link"/>
-      <child link="base_footprint" />
-    </joint>
     <joint name="wheel_left_joint" type="continuous">
       <parent link="base_link"/>

File: kobuki_description/urdf/kobuki_gazebo.urdf.xacro (robot description, xacro)
@@ -46,5 +46,4 @@
 	    </sensor>
 	  </gazebo>
-    <!--
 	  <gazebo reference="cliff_sensor_left_link">
 	    <sensor type="ray" name="cliff_sensor_left">
@@ -57,8 +56,8 @@
 	            <samples>50</samples>
 	            <resolution>1.0</resolution>
-	            <min_angle>-0.0436</min_angle>
-	            <max_angle>0.0436</max_angle>
+	            <min_angle>-0.0436</min_angle>  <!-- -2.5 degree -->
+	            <max_angle>0.0436</max_angle> <!-- 2.5 degree -->
 	          </horizontal>
-           Can't use vertical rays until this bug is resolved: -->
+<!--            Can't use vertical rays until this bug is resolved: -->
 <!--            https://bitbucket.org/osrf/gazebo/issue/509/vertical-sensor-doesnt-works -->
 <!-- 	          <vertical> -->
@@ -67,5 +66,5 @@
 <!-- 	            <min_angle>-0.0436</min_angle>  -2.5 degree -->
 <!-- 	            <max_angle>0.0436</max_angle> 2.5 degree -->
-<!-- 	          </vertical>
+<!-- 	          </vertical> -->
 	        </scan>
 	        <range>
@@ -77,6 +76,4 @@
 	    </sensor>
 	  </gazebo>
-    -->
-    <!--
 	  <gazebo reference="cliff_sensor_right_link">
 	    <sensor type="ray" name="cliff_sensor_right">
@@ -89,8 +86,8 @@
 	            <samples>50</samples>
 	            <resolution>1.0</resolution>
-	            <min_angle>-0.0436</min_angle>
-	            <max_angle>0.0436</max_angle>
+	            <min_angle>-0.0436</min_angle>  <!-- -2.5 degree -->
+	            <max_angle>0.0436</max_angle> <!-- 2.5 degree -->
 	          </horizontal>
-           Can't use vertical rays until this bug is resolved: -->
+<!--            Can't use vertical rays until this bug is resolved: -->
 <!--            https://bitbucket.org/osrf/gazebo/issue/509/vertical-sensor-doesnt-works -->
 <!-- 	          <vertical> -->
@@ -99,5 +96,5 @@
 <!-- 	            <min_angle>-0.0436</min_angle>  -2.5 degree -->
 <!-- 	            <max_angle>0.0436</max_angle> 2.5 degree -->
-<!-- 	          </vertical>
+<!-- 	          </vertical> -->
 	        </scan>
 	        <range>
@@ -109,6 +106,4 @@
 	    </sensor>
 	  </gazebo>
-    -->
-    <!--
 	  <gazebo reference="cliff_sensor_front_link">
 	    <sensor type="ray" name="cliff_sensor_front">
@@ -121,8 +116,8 @@
 	            <samples>50</samples>
 	            <resolution>1.0</resolution>
-	            <min_angle>-0.0436</min_angle>
-	            <max_angle>0.0436</max_angle> <
+	            <min_angle>-0.0436</min_angle>  <!-- -2.5 degree -->
+	            <max_angle>0.0436</max_angle> <!-- 2.5 degree -->
 	          </horizontal>
-	          Can't use vertical rays until this bug is resolved: -->
+<!-- 	          Can't use vertical rays until this bug is resolved: -->
 <!--            https://bitbucket.org/osrf/gazebo/issue/509/vertical-sensor-doesnt-works -->
 <!-- 	          <vertical> -->
@@ -131,5 +126,5 @@
 <!-- 	            <min_angle>-0.0436</min_angle>  -2.5 degree -->
 <!-- 	            <max_angle>0.0436</max_angle> 2.5 degree -->
-<!-- 	          </vertical>
+<!-- 	          </vertical> -->
 	        </scan>
 	        <range>
@@ -141,5 +136,4 @@
 	    </sensor>
 	  </gazebo>
-  -->
 	  <gazebo reference="gyro_link">
 	   <sensor type="imu" name="imu">
@@ -160,9 +154,9 @@
 	          <rate>
 	            <mean>0.0</mean>
-	            <stddev>${0.0014*0.0014}</stddev>
+	            <stddev>${0.0014*0.0014}</stddev> <!-- 0.25 x 0.25 (deg/s) -->
 	            <bias_mean>0.0</bias_mean>
 	            <bias_stddev>0.0</bias_stddev>
 	          </rate>
-		        <accel>
+		        <accel> <!-- not used in the plugin and real robot, hence using tutorial values -->
 			        <mean>0.0</mean>
 			        <stddev>1.7e-2</stddev>
@@ -176,5 +170,5 @@
 	  <gazebo>
 	    <plugin name="differential_drive_controller" filename="libgazebo_ros_diff_drive.so">
-        <update_rate>10</update_rate>
+    		<update_rate>10</update_rate>
         <left_joint>wheel_left_joint</left_joint>
         <right_joint>wheel_right_joint</right_joint>
